File: Hardware/Laser Driver/Sch.sch (EAGLE design)
At the start: 33 parts, among them IC1 LMH6645MF

Commit message: Added hardware and software files
Parts:
- removed R14: 1R, SparkFun-Passives:RESISTOR0603-RES
- added C1: 100n, SparkFun-Passives:CAP1206
- added C6: 15u, SparkFun-Passives:CAP1206
- added C7: 10u, SparkFun-Passives:CAP1206
- added JP6: (no value), SparkFun-Connectors:M04PTH
- added R1: 5k, resistor:R-TRIMM64W
- added R15: 1R, EagleParts:CRM2010-JW-1R0ELF
- added R2: 240R, SparkFun-Passives:RESISTOR0603-RES
- added U1: TL1963ADCQR, EagleParts:TL1963ADCQR
- C5: value 47u -> 15u
- R11: device SparkFun-Passives:RESISTORAXIAL-0.3 -> resistor:R-US_R0603
- R12, R3: device pot:TRIM_EU-CA9V -> resistor:R-TRIMM5X
- R4: value (none) -> 22k
- TP1, TP2, TP3, TP4, TP7, TP8, TP9: device SparkFun-Connectors:M01PTH_LONGPAD -> SparkFun-Connectors:M01PTH
Connections:
- removed net N$1: R12.E, TP1.1
- new net +12V: C7.1, JP6.2, U1.!SHDN, U1.IN
- new net BRIGHTNESS: D2.AC, JP6.4, R12.E, TP1.1
- new net N$16: R1.E, R2.2, U1.SENSE/ADJ
- net +5V: now also JP6.3
- net GNDA: now also C6.2, C7.2, JP6.1, R15.R2, R2.1, U1.GND, U1.GND_2; no longer R14.1
- net N$14: now also C1.1
- net N$15: now also R15.R1; no longer R14.2
- net N$2: no longer D2.AC
- net VCC: now also C1.2, C6.1, R1.S, U1.OUT
Other:
- moved on the sheet: D2, TP9
